Commit message: Edited the Urdf file for floor 1

File: urdf/btechbot.urdf (robot description, URDF)
Before this commit: robot btechbot, 3 links, 2 joints
Links:
- removed link left wheel
- removed link right wheel
- added link chassis; visual box size=0.22 0.18 0.003
- added link column1.1; visual cylinder length=0.05 radius=0.0025
- added link column1.2; visual cylinder length=0.05 radius=0.0025
- added link column1.3; visual cylinder length=0.05 radius=0.0025
- added link column1.4; visual cylinder length=0.05 radius=0.0025
- added link floor1; visual cylinder length=0.003 radius=0.075
- added link left_wheel; visual cylinder length=0.018 radius=0.022
- added link right_wheel; visual cylinder length=0.018 radius=0.022
- link base_link: geometry 
Joints:
- added joint chassis_joint: type fixed, parent base_link, child chassis, origin xyz=0 0 0
- added joint column1.1: type fixed, parent chassis, child column1.1, origin xyz=0.055 0 0 rpy=0 0 0
- added joint column1.2: type fixed, parent chassis, child column1.2, origin xyz=-0.055 0 0 rpy=0 0 0
- added joint column1.3: type fixed, parent chassis, child column1.3, origin xyz=0 -0.045 0 rpy=0 0 0
- added joint column1.4: type fixed, parent chassis, child column1.4, origin xyz=0 0.045 0 rpy=0 0 0
- added joint floor1.1: type fixed, parent column1.1, child floor1, origin xyz=-0.055 0 0.0515 rpy=0 0 0
- added joint floor1.2: type fixed, parent column1.2, child floor1, origin xyz=0.055 0 0.0515 rpy=0 0 0
- added joint floor1.3: type fixed, parent column1.3, child floor1, origin xyz=0 -0.045 0.0515 rpy=0 0 0
- added joint floor1.4: type fixed, parent column1.4, child floor1, origin xyz=0 -0.045 0.0515 rpy=0 0 0
- joint lwheel: axis 0 1 0 -> 0 0 -1; child left wheel -> left_wheel; origin xyz=0 0 0 rpy=1.587 0 0 -> xyz=0 0.099 0 rpy=1.587 0 0
- joint rwheel: axis 0 1 0 -> 0 0 1; child right wheel -> right_wheel; origin xyz=0 0 0 rpy=1.587 0 0 -> xyz=0 -0.099 0 rpy=-1.587 0 0

Commit message: Added Floor2

File: urdf/btechbot.urdf (robot description, URDF)
Before this commit: robot btechbot, 9 links, 11 joints
Links:
- added link column2.1; visual cylinder length=0.05 radius=0.0025
- added link column2.2; visual cylinder length=0.05 radius=0.0025
- added link column2.3; visual cylinder length=0.05 radius=0.0025
- added link column2.4; visual cylinder length=0.05 radius=0.0025
- added link floor2; visual cylinder length=0.003 radius=0.075
Joints:
- added joint column2.1: type fixed, parent floor1, child column2.1, origin xyz=0.055 0 0.025 rpy=0 0 0
- added joint column2.2: type fixed, parent floor1, child column2.2, origin xyz=-0.055 0 0.025 rpy=0 0 0
- added joint column2.3: type fixed, parent floor1, child column2.3, origin xyz=0 -0.045 0.025 rpy=0 0 0
- added joint column2.4: type fixed, parent floor1, child column2.4, origin xyz=0 0.045 0.025 rpy=0 0 0
- added joint floor2.1: type fixed, parent column2.1, child floor2, origin xyz=-0.055 0 0.025 rpy=0 0 0
- added joint floor2.2: type fixed, parent column2.2, child floor2, origin xyz=0.055 0 0.025 rpy=0 0 0
- added joint floor2.3: type fixed, parent column2.3, child floor2, origin xyz=0 -0.045 0.025 rpy=0 0 0
- added joint floor2.4: type fixed, parent column2.4, child floor2, origin xyz=0 -0.045 0.025 rpy=0 0 0
- joint column1.1: origin xyz=0.055 0 0 rpy=0 0 0 -> xyz=0.055 0 0.025 rpy=0 0 0
- joint column1.2: origin xyz=-0.055 0 0 rpy=0 0 0 -> xyz=-0.055 0 0.025 rpy=0 0 0
- joint column1.3: origin xyz=0 -0.045 0 rpy=0 0 0 -> xyz=0 -0.045 0.025 rpy=0 0 0
- joint column1.4: origin xyz=0 0.045 0 rpy=0 0 0 -> xyz=0 0.045 0.025 rpy=0 0 0
- joint floor1.1: origin xyz=-0.055 0 0.0515 rpy=0 0 0 -> xyz=-0.055 0 0.025 rpy=0 0 0
- joint floor1.2: origin xyz=0.055 0 0.0515 rpy=0 0 0 -> xyz=0.055 0 0.025 rpy=0 0 0
- joint floor1.3: origin xyz=0 -0.045 0.0515 rpy=0 0 0 -> xyz=0 -0.045 0.025 rpy=0 0 0
- joint floor1.4: origin xyz=0 -0.045 0.0515 rpy=0 0 0 -> xyz=0 -0.045 0.025 rpy=0 0 0

Commit message: added collision to the urdf file

File: urdf/btechbot.urdf (robot description, URDF)
Before this commit: robot btechbot, 14 links, 19 joints
Links:
- added link bcaster; collision sphere radius=0.022; visual sphere radius=0.022
- added link fcaster; collision sphere radius=0.022; visual sphere radius=0.022
- link chassis: geometry collision box size=0.22 0.18 0.003; visual box size=0.22 0.18 0.003
- link column1.1: geometry collision cylinder length=0.05 radius=0.0025; visual cylinder length=0.05 radius=0.0025
- link column1.2: geometry collision cylinder length=0.05 radius=0.0025; visual cylinder length=0.05 radius=0.0025
- link column1.3: geometry collision cylinder length=0.05 radius=0.0025; visual cylinder length=0.05 radius=0.0025
- link column1.4: geometry collision cylinder length=0.05 radius=0.0025; visual cylinder length=0.05 radius=0.0025
- link column2.1: geometry collision cylinder length=0.05 radius=0.0025; visual cylinder length=0.05 radius=0.0025
- link column2.2: geometry collision cylinder length=0.05 radius=0.0025; visual cylinder length=0.05 radius=0.0025
- link column2.3: geometry collision cylinder length=0.05 radius=0.0025; visual cylinder length=0.05 radius=0.0025
- link column2.4: geometry collision cylinder length=0.05 radius=0.0025; visual cylinder length=0.05 radius=0.0025
- link floor1: geometry collision cylinder length=0.003 radius=0.075; visual cylinder length=0.003 radius=0.075
- link floor2: geometry collision cylinder length=0.003 radius=0.075; visual cylinder length=0.003 radius=0.075
- link left_wheel: geometry collision cylinder length=0.018 radius=0.022; visual cylinder length=0.018 radius=0.022
- link right_wheel: geometry collision cylinder length=0.018 radius=0.022; visual cylinder length=0.018 radius=0.022
Joints:
- added joint bcaster: type continuous, parent base_link, child bcaster, origin xyz=-0.0775 0 0 rpy=0 0 0, axis 1 1 1
- added joint fcaster: type continuous, parent base_link, child fcaster, origin xyz=0.0775 0 0 rpy=0 0 0, axis 1 1 1

Commit message: added inertial tags

File: urdf/btechbot.urdf (robot description, URDF)
Before this commit: robot btechbot, 16 links, 21 joints
Links:
- link bcaster: mass None -> 0.015
- link chassis: mass None -> 0.05
- link column1.1: mass None -> 0.01
- link column1.2: mass None -> 0.01
- link column1.3: mass None -> 0.01
- link column1.4: mass None -> 0.01
- link column2.1: mass None -> 0.01
- link column2.2: mass None -> 0.01
- link column2.3: mass None -> 0.01
- link column2.4: mass None -> 0.01
- link fcaster: mass None -> 0.015
- link floor1: mass None -> 0.04
- link floor2: mass None -> 0.04
- link left_wheel: mass None -> 0.018
- link right_wheel: mass None -> 0.018

Commit message: Modified the URDF for Gazebo, created an empty world gazebo launch file that spawns the btechbot

File: urdf/btechbot.urdf (robot description, URDF)
Before this commit: robot btechbot, 16 links, 21 joints
Links:
- removed link bcaster
- removed link column1.1
- removed link column1.2
- removed link column1.3
- removed link column1.4
- removed link column2.1
- removed link column2.2
- removed link column2.3
- removed link column2.4
- removed link fcaster
- added link back_caster, mass 0.015; collision sphere radius=0.022; visual sphere radius=0.022
- added link column1_1, mass 0.01; collision cylinder length=0.05 radius=0.0025; visual cylinder length=0.05 radius=0.0025
- added link column1_2, mass 0.01; collision cylinder length=0.05 radius=0.0025; visual cylinder length=0.05 radius=0.0025
- added link column1_3, mass 0.01; collision cylinder length=0.05 radius=0.0025; visual cylinder length=0.05 radius=0.0025
- added link column1_4, mass 0.01; collision cylinder length=0.05 radius=0.0025; visual cylinder length=0.05 radius=0.0025
- added link column2_1, mass 0.01; collision cylinder length=0.05 radius=0.0025; visual cylinder length=0.05 radius=0.0025
- added link column2_2, mass 0.01; collision cylinder length=0.05 radius=0.0025; visual cylinder length=0.05 radius=0.0025
- added link column2_3, mass 0.01; collision cylinder length=0.05 radius=0.0025; visual cylinder length=0.05 radius=0.0025
- added link column2_4, mass 0.01; collision cylinder length=0.05 radius=0.0025; visual cylinder length=0.05 radius=0.0025
- added link front_caster, mass 0.015; collision sphere radius=0.022; visual sphere radius=0.022
Joints:
- removed joint floor1.2
- removed joint floor1.3
- removed joint floor1.4
- removed joint floor2.1
- removed joint floor2.3
- removed joint floor2.4
- joint bcaster: axis 1 1 1 -> (none); child bcaster -> back_caster; type continuous -> fixed
- joint column1.1: child column1.1 -> column1_1
- joint column1.2: child column1.2 -> column1_2
- joint column1.3: child column1.3 -> column1_3
- joint column1.4: child column1.4 -> column1_4
- joint column2.1: child column2.1 -> column2_1
- joint column2.2: child column2.2 -> column2_2
- joint column2.3: child column2.3 -> column2_3
- joint column2.4: child column2.4 -> column2_4
- joint fcaster: axis 1 1 1 -> (none); child fcaster -> front_caster; type continuous -> fixed
- joint floor1.1: parent column1.1 -> column1_1
- joint floor2.2: parent column2.2 -> column2_2
