Commit message: Added Lidar, LaserScan, obstacles world

File: urdf/btechbot.urdf.xacro (robot description, xacro)
@@ -3,3 +3,4 @@
 <xacro:include filename="btechbot_core.xacro"/>
 <xacro:include filename="btechbot_control.xacro"/>
+<xacro:include filename="lidar.xacro"/>
 </robot>

File: urdf/btechbot_core.xacro (robot description, xacro)
@@ -441,4 +441,29 @@
    <origin xyz = "0.055 0 0.025" rpy = "0 0 0" />
  </joint>
+ <joint name="laser_joint" type="fixed">
+  <parent link="floor2"/>
+  <child link="laser_frame"/>
+  <origin xyz="0 0 0.022" rpy="0 0 0"/>
+</joint>
+<link name="laser_frame">
+  <visual>
+      <geometry>
+        <cylinder radius = "0.022" length = "0.018" />
+      </geometry>
+      <material name = "blue">
+        <color rgba = "0.1 0.1 1.0 1.0"/>
+      </material>
+   </visual>
+   <collision>
+      <geometry>
+        <cylinder radius = "0.022" length = "0.018" />
+      </geometry>
+   </collision>
+   <inertial>
+      <mass value = "0.018" />
+      <origin xyz = "0 0 0" rpy = "0 0 0" />
+      <inertia ixx = "0.0002" ixz = "0" ixy="0" iyy = "0.0002" iyz = "0" izz = "0.00004" />
+    </inertial>
+</link>
  <!--joint name = "floor2.3" type = "fixed">
    <parent link = "column2_3" />
@@ -482,4 +507,33 @@
  </gazebo>
 	 -->
+<gazebo reference="laser_frame">
+	<sensor name="laser" type="ray">
+		<pose>0 0 0 0 0 0</pose>
+		<visualize>true</visualize>
+		<update_rate>10</update_rate>
+		<ray>
+			<scan>
+			<horizontal>
+				<samples>360</samples>
+				<resolution>1</resolution>
+				<min_angle>-3.14</min_angle>
+				<max_angle>3.14</max_angle>
+			</horizontal>
+			</scan>
+			<range>
+				<min>0.3</min>
+				<max>12</max>
+				<resolution>0.01</resolution>
+			</range>
+		</ray>
+		<plugin name="laser_contrller" filename="libgazebo_ros_laser.so">
+			<ros>
+				<argument>=~/out:=scan</argument>
+			</ros>
+			<topicName>sensor_msgs/LaserScan</topicName>
+			<frameName>laser_frame</frameName>
+		</plugin>
+	</sensor>
+</gazebo>
 <gazebo>
 	<plugin name="diff_drive_btechbot" filename="libgazebo_ros_diff_drive.so">

Commit message: Added Slam_toolbox, Basic_onlieAsync Slam working, needs to be tweaked

File: urdf/btechbot.urdf.xacro (robot description, xacro)
@@ -4,3 +4,4 @@
 <xacro:include filename="btechbot_control.xacro"/>
 <xacro:include filename="lidar.xacro"/>
+<!--xacro:include filename="ros_control.xacro"/-->
 </robot>

File: urdf/btechbot_control.xacro (robot description, xacro)
@@ -2,5 +2,5 @@
 <robot xmlns:xacro="http://www.ros.org/wiki/xacro">
 <gazebo>
-<plugin name="diff_drive_btechbot" filename="libgazebo_ros_diffdrive.so">
+	<plugin name="diff_drive_btechbot" filename="libgazebo_ros_diffdrive.so">
 		<left_joint>lwheel</left_joint>
 		<right_joint>rwheel</right_joint>
@@ -14,5 +14,5 @@
 		<publish_odom_tf>true</publish_odom_tf>
 		<publish_wheel_tf>true</publish_wheel_tf>
-</plugin>
+	</plugin>
 </gazebo>
 </robot>

File: urdf/btechbot_core.xacro (robot description, xacro)
@@ -507,4 +507,5 @@
  </gazebo>
 	 -->
+<!-- LiDAR setup for gazbeo -->
 <gazebo reference="laser_frame">
 	<sensor name="laser" type="ray">
@@ -515,5 +516,5 @@
 			<scan>
 			<horizontal>
-				<samples>360</samples>
+				<samples>359</samples>
 				<resolution>1</resolution>
 				<min_angle>-3.14</min_angle>
@@ -527,5 +528,5 @@
 			</range>
 		</ray>
-		<plugin name="laser_contrller" filename="libgazebo_ros_laser.so">
+		<plugin name="laser_controller" filename="libgazebo_ros_laser.so">
 			<ros>
 				<argument>=~/out:=scan</argument>
@@ -536,4 +537,32 @@
 	</sensor>
 </gazebo>
+<!--ROS_CONTROL SETUP-->
+<!--ros_control name="GazeboBtechbot" type="system">
+	<hardware>
+		<plugin>gazebo_ros_control/GazeboBtechbot</plugin>
+	</hardware>
+	<joint name="lwheel">
+		<command_interface name="velocity">
+			<param name="min">-10</param>
+			<param name="max">10</param>
+		</command_interface>
+		<state_interface name="velocity"/>
+		<state_interface name="position"/>
+	</joint>
+	<joint name="rwheel">
+		<command_interface name="velocity">
+			<param name="min">-10</param>
+			<param name="max">10</param>
+		</command_interface>
+		<state_interface name="velocity"/>
+		<state_interface name="position"/>
+	</joint>
+</ros_control>
+<gazebo>
+	<plugin name="gazebo_btechbot_control" filename="libgazebo_ros_control.so">
+		<parameters>$(find btechbot)/config/controllers.yaml</parameters>
+	</plugin>
+</gazebo-->
+<!--Working libgazebo_diff_drive.so  controller setup-->
 <gazebo>
 	<plugin name="diff_drive_btechbot" filename="libgazebo_ros_diff_drive.so">
